File: hairio_full_3/drive_board.brd (EAGLE design)
At the start: 68.2 x 54.6 mm, 29 parts, among them J1 105313-1104, J2 105313-1104, P1 S2B-PH-SM4-TB(LF)(SN), P2 S2B-PH-SM4-TB(LF)(SN)

Commit message: updated board files
Parts:
- moved P2 5.84 mm to (81.2, 68.1)
- moved JP1 3.70 mm to (80.3, 58.2), turned to 270 degrees
- moved PNP1 0.52 mm to (52.6, 45.6)
- moved J1 0.28 mm to (43.3, 27.7)
Routing:
- net N$12: track 18.5 -> 10.8 mm
- net DRIVE_SIGNAL_2: track 32.3 -> 34.2 mm
- net N$4: track 29.9 -> 31.8 mm
- net D6: track 7.08 -> 8.53 mm
- net N$13: track 37.4 -> 38.4 mm
- net N$8: track 22.8 -> 23.7 mm
- net GND: track 44.8 -> 45.6 mm
- net N$16: track 8.26 -> 7.41 mm
- net CAPTOUCH_2: track 66.6 -> 65.8 mm
- net CAPTOUCH_1: track 46.1 -> 45.4 mm
- net A2_THERM_2: track 58.7 -> 58.2 mm
Other:
- board size 68.2 x 54.6 mm -> 58 x 49 mm
